File: pcb/rc.sch (EAGLE design)
At the start: 57 parts, among them IC2 TP4056

Commit message: scheme: change H-bridge and battety check
Parts:
- removed MA, MB: WIREPADSMD5-2,5, wirepad:WIREPADSMD5-2,5
- removed Q1: (no value), semicon-smd-ipc:PNP-TRANSISTOR_SOT23
- removed R14: (no value), skydrop:R_0805
- added D2, D3, D4, D5: (no value), skydrop:DIODESMA
- added MOTOR_A, MOTOR_B: WIREPADSMD5-2,5, wirepad:WIREPADSMD5-2,5
- added T10, T11: (no value), zetex:NPNSOT23
Connections:
- removed net H_LN: R5.2, U1.GPIO12
- removed net H_LP: R4.2, U1.GPIO13
- removed net H_RN: R6.1, U1.GPIO5
- removed net H_RP: R3.1, U1.GPIO14
- new net BAT_CHECK: T11.C, U1.GPIO12
- new net H_BCK: R3.1, U1.GPIO13
- new net H_FWD: R4.2, U1.GPIO14
- new net H_PWM: R5.2, U1.GPIO5
- new net N$31: D4.C, D5.C, T10.C
- new net N$32: R5.1, T10.B
- net BAT_PROT: now also R10.1, R2.1
- net GND: now also T10.E, T11.E; no longer R10.1, R2.1
- net N$1: now also D2.C
- net N$10: no longer Q1.E
- net N$13: now also R6.2, T11.B; no longer Q1.B, R14.1
- net N$17: now also R6.1; no longer R14.2
- net N$24: no longer Q1.C
- net N$3: now also MOTOR_A.P; no longer MA.P
- net N$4: now also MOTOR_B.P; no longer MB.P
- net N$6: now also D2.A, D4.A; no longer R5.1
- net N$8: now also D3.C
- net N$9: now also D3.A, D5.A; no longer R6.2
Other:
- moved on the sheet: R1, R10, R13, R2, R3, R4, R5, R6, R9, T1, T2, T3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

Commit message: begin pcb v2
Parts:
- removed CHAGER+, CHARGER-: WIREPADSMD5-2,5, wirepad:WIREPADSMD5-2,5
- removed D1, D5: (no value), skydrop:DIODESMA
- added D6: (no value), skydrop:DIODE_SOD-123FL
- added J1: (no value), skydrop:USB-AB
- added R14: 0, skydrop:R_1206
- added R24: (no value), skydrop:R_1206
- D2, D3, D4: device skydrop:DIODESMA -> skydrop:DIODE_SOD-123FL
Connections:
- net N$14 renamed BAT+
- net N$15 renamed TX
- net N$18 renamed RX
- removed net N$10: IC1.VCC, IC2.BAT, R8.1, T7.S, T9.S
- removed net N$24: D1.C, R13.1, T9.G
- new net BAT_CHRG: IC2.BAT, R8.1, T7.S, T9.S
- new net N$14: R14.1, T11.C
- net BAT_CHECK: now also R14.2; no longer T11.C
- net BAT_PROT: now also IC1.VCC
- net GND: now also J1.GND; no longer CHARGER-.P
- net N$31: now also D6.C; no longer D5.C
- net N$9: now also D6.A; no longer D5.A
- net V_CHRG: now also J1.VBUS, R13.1, R24.1, R24.2, T9.G; no longer CHAGER+.P, D1.A
Other:
- moved on the sheet: BAT+, BAT-, IC1, R13, R6, T11, T9

Commit message: pcb
Parts:
- added GND19, GND20: WIREPADSMD5-1,8, wirepad:WIREPADSMD5-1,8
- R24: value (none) -> 0
Connections:
- new net N$10: C2.1, J1.VBUS, R24.2
- net GND: now also GND20.P
- net N$21: now also GND19.P
- net V_CHRG: no longer C2.1, J1.VBUS, R24.2
Other:
- moved on the sheet: D2, D3, D4, D6, MOTOR_A, MOTOR_B, R1, R10, R2, R24, R3, R4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

Commit message: pcb
Parts:
- added JP1, JP2, JP5: (no value), adafruit:PINHD-1X3
- added JP3, JP4: (no value), adafruit:PINHD-1X1
- renumbered GND19 to FLASH1, GND20 to FLASH2
Changed lines of the file:
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@@
 <part name="R14" library="skydrop" deviceset="R_" device="1206" value="0"/>
 <part name="R24" library="skydrop" deviceset="R_" device="1206" value="0"/>
-<part name="GND19" library="wirepad" library_urn="urn:adsk.eagle:library:412" deviceset="WIREPAD" device="SMD5-1,8" package3d_urn="urn:adsk.eagle:package:30844/1" value="WIREPADSMD5-1,8"/>
-<part name="GND20" library="wirepad" library_urn="urn:adsk.eagle:library:412" deviceset="WIREPAD" device="SMD5-1,8" package3d_urn="urn:adsk.eagle:package:30844/1" value="WIREPADSMD5-1,8"/>
+<part name="FLASH1" library="wirepad" library_urn="urn:adsk.eagle:library:412" deviceset="WIREPAD" device="SMD5-1,8" package3d_urn="urn:adsk.eagle:package:30844/1" value="WIREPADSMD5-1,8"/>
+<part name="FLASH2" library="wirepad" library_urn="urn:adsk.eagle:library:412" deviceset="WIREPAD" device="SMD5-1,8" package3d_urn="urn:adsk.eagle:package:30844/1" value="WIREPADSMD5-1,8"/>
 <part name="GND21" library="supply1" library_urn="urn:adsk.eagle:library:371" deviceset="GND" device=""/>
+<part name="JP1" library="adafruit" deviceset="PINHD-1X3" device=""/>
+<part name="JP2" library="adafruit" deviceset="PINHD-1X3" device=""/>
+<part name="JP5" library="adafruit" deviceset="PINHD-1X3" device=""/>
+<part name="JP3" library="adafruit" deviceset="PINHD-1X1" device=""/>
+<part name="JP4" library="adafruit" deviceset="PINHD-1X1" device=""/>
 </parts>
 <sheets>
@@
 <instance part="R14" gate="G$1" x="137.16" y="20.32" rot="R90"/>
 <instance part="R24" gate="G$1" x="177.8" y="96.52"/>
-<instance part="GND19" gate="G$1" x="129.54" y="129.54" rot="MR0"/>
-<instance part="GND20" gate="G$1" x="129.54" y="127" rot="MR0"/>
+<instance part="FLASH1" gate="G$1" x="129.54" y="129.54" smashed="yes" rot="MR0">
+<attribute name="NAME" x="130.683" y="131.3942" size="1.778" layer="95" rot="MR0"/>
+<attribute name="VALUE" x="130.683" y="126.238" size="1.778" layer="96" rot="MR0"/>
+</instance>
+<instance part="FLASH2" gate="G$1" x="129.54" y="127" rot="MR0"/>
 <instance part="GND21" gate="1" x="124.46" y="119.38" rot="MR0"/>
+<instance part="JP1" gate="A" x="165.1" y="137.16"/>
+<instance part="JP2" gate="A" x="266.7" y="160.02"/>
+<instance part="JP5" gate="A" x="195.58" y="137.16"/>
+<instance part="JP3" gate="G$1" x="167.64" y="119.38"/>
+<instance part="JP4" gate="G$1" x="167.64" y="114.3"/>
 </instances>
 <busses>
@@
 <segment>
 <pinref part="GND21" gate="1" pin="GND"/>
-<pinref part="GND20" gate="G$1" pin="P"/>
+<pinref part="FLASH2" gate="G$1" pin="P"/>
 <wire x1="124.46" y1="121.92" x2="124.46" y2="127" width="0.1524" layer="91"/>
 <wire x1="124.46" y1="127" x2="127" y2="127" width="0.1524" layer="91"/>
@@
 <pinref part="U1" gate="G$1" pin="GPIO0"/>
 <wire x1="109.22" y1="129.54" x2="93.98" y2="129.54" width="0.1524" layer="91"/>
-<pinref part="GND19" gate="G$1" pin="P"/>
+<pinref part="FLASH1" gate="G$1" pin="P"/>
 <wire x1="127" y1="129.54" x2="109.22" y2="129.54" width="0.1524" layer="91"/>
 <junction x="109.22" y="129.54"/>
@@
 <segment>
 <pinref part="R5" gate="G$1" pin="2"/>
-<wire x1="-48.26" y1="-27.94" x2="-53.34" y2="-12.7" width="0.1524" layer="91"/>
-<label x="-63.5" y="-12.7" size="1.778" layer="95"/>
-</segment>
-</net>
+<wire x1="-48.26" y1="-27.94" x2="-55.88" y2="-27.94" width="0.1524" layer="91"/>
+<label x="-60.96" y="-22.86" size="1.778" layer="95"/>
+</segment>
+</net>

Commit message: pcb
Parts:
- added C7: (no value), skydrop:C-EUC0805
- added C8, C9: (no value), adafruit:CPOL-USD/7343-31W
- added D5: (no value), adafruit:DIODESMA
- added IC4: (no value), my:NCP1450A
- added L1: (no value), inductor-neosid:MS85
- added R25: 0, skydrop:R_1206
- added T12: (no value), zetex:NMOSSOT23
- IC2: device TP4056:TP4056 -> my:TP4056
Connections:
- new net N$15: IC4.EXT, T12.G
- new net N$18: IC4.CE, R25.1
- new net N$24: C9.+, L1.1, R25.2
- new net N$3: D5.A, L1.2, T12.D
- new net N$34: C7.2, C8.+, D5.C, IC4.OUT
- net GND: now also C7.1, C8.-, C9.-, IC2.HEATSINK, IC4.GND, T12.S
Other:
- moved on the sheet: LED1, R21
Changed lines of the file:
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@@
 <part name="IC1" library="skydrop" deviceset="TCM809" device=""/>
 <part name="T8" library="zetex" library_urn="urn:adsk.eagle:library:418" deviceset="NPNSOT23" device="" package3d_urn="urn:adsk.eagle:package:30981/1"/>
-<part name="IC2" library="TP4056" deviceset="TP4056" device=""/>
+<part name="IC2" library="my" deviceset="TP4056" device=""/>
 <part name="R8" library="skydrop" deviceset="R_" device="0805"/>
 <part name="GND8" library="supply1" library_urn="urn:adsk.eagle:library:371" deviceset="GND" device=""/>
@@
 <part name="JP3" library="adafruit" deviceset="PINHD-1X1" device=""/>
 <part name="JP4" library="adafruit" deviceset="PINHD-1X1" device=""/>
+<part name="GND19" library="supply1" library_urn="urn:adsk.eagle:library:371" deviceset="GND" device=""/>
+<part name="IC4" library="my" deviceset="NCP1450A" device=""/>
+<part name="D5" library="adafruit" deviceset="DIODE" device="SMA"/>
+<part name="L1" library="inductor-neosid" library_urn="urn:adsk.eagle:library:241" deviceset="MS85" device="" package3d_urn="urn:adsk.eagle:package:14698/1"/>
+<part name="T12" library="zetex" library_urn="urn:adsk.eagle:library:418" deviceset="NMOSSOT23" device="" package3d_urn="urn:adsk.eagle:package:30981/1"/>
+<part name="GND20" library="supply1" library_urn="urn:adsk.eagle:library:371" deviceset="GND" device=""/>
+<part name="C7" library="skydrop" deviceset="C-EU" device="C0805"/>
+<part name="GND22" library="supply1" library_urn="urn:adsk.eagle:library:371" deviceset="GND" device=""/>
+<part name="C8" library="adafruit" deviceset="CPOL-US" device="D/7343-31W"/>
+<part name="C9" library="adafruit" deviceset="CPOL-US" device="D/7343-31W"/>
+<part name="GND23" library="supply1" library_urn="urn:adsk.eagle:library:371" deviceset="GND" device=""/>
+<part name="GND24" library="supply1" library_urn="urn:adsk.eagle:library:371" deviceset="GND" device=""/>
+<part name="R25" library="skydrop" deviceset="R_" device="1206" value="0"/>
 </parts>
 <sheets>
@@
 <instance part="C2" gate="G$1" x="241.3" y="91.44"/>
 <instance part="C3" gate="G$1" x="241.3" y="58.42"/>
-<instance part="R21" gate="G$1" x="195.58" y="68.58" rot="MR180"/>
-<instance part="LED1" gate="G$1" x="203.2" y="76.2"/>
+<instance part="R21" gate="G$1" x="198.12" y="68.58" rot="MR180"/>
+<instance part="LED1" gate="G$1" x="205.74" y="76.2"/>
 <instance part="IC3" gate="G1" x="12.7" y="116.84"/>
 <instance part="GND13" gate="1" x="15.24" y="96.52"/>
@@
 <instance part="JP3" gate="G$1" x="167.64" y="119.38"/>
 <instance part="JP4" gate="G$1" x="167.64" y="114.3"/>
+<instance part="GND19" gate="1" x="175.26" y="53.34"/>
+<instance part="IC4" gate="G1" x="-88.9" y="109.22"/>
+<instance part="D5" gate="G$1" x="-63.5" y="129.54"/>
+<instance part="L1" gate="G$1" x="-81.28" y="129.54"/>
+<instance part="T12" gate="A" x="-71.12" y="116.84"/>
+<instance part="GND20" gate="1" x="-71.12" y="93.98"/>
+<instance part="C7" gate="G$1" x="-106.68" y="101.6" rot="R180"/>
+<instance part="GND22" gate="1" x="-106.68" y="93.98"/>
+<instance part="C8" gate="G$1" x="-48.26" y="109.22"/>
+<instance part="C9" gate="G$1" x="-121.92" y="109.22"/>
+<instance part="GND23" gate="1" x="-121.92" y="93.98"/>
+<instance part="GND24" gate="1" x="-48.26" y="93.98"/>
+<instance part="R25" gate="G$1" x="-101.6" y="121.92" rot="R90"/>
 </instances>
 <busses>
@@
 <wire x1="124.46" y1="121.92" x2="124.46" y2="127" width="0.1524" layer="91"/>
 <wire x1="124.46" y1="127" x2="127" y2="127" width="0.1524" layer="91"/>
+</segment>
+<segment>
+<pinref part="IC2" gate="G$1" pin="HEATSINK"/>
+<pinref part="GND19" gate="1" pin="GND"/>
+<wire x1="175.26" y1="60.96" x2="175.26" y2="55.88" width="0.1524" layer="91"/>
+</segment>
+<segment>
+<pinref part="IC4" gate="G1" pin="GND"/>
+<wire x1="-78.74" y1="104.14" x2="-71.12" y2="104.14" width="0.1524" layer="91"/>
+<pinref part="T12" gate="A" pin="S"/>
+<wire x1="-71.12" y1="104.14" x2="-71.12" y2="111.76" width="0.1524" layer="91"/>
+<pinref part="GND20" gate="1" pin="GND"/>
+<wire x1="-71.12" y1="96.52" x2="-71.12" y2="104.14" width="0.1524" layer="91"/>
+<junction x="-71.12" y="104.14"/>
+</segment>
+<segment>
+<pinref part="GND22" gate="1" pin="GND"/>
+<pinref part="C7" gate="G$1" pin="1"/>
+<wire x1="-106.68" y1="96.52" x2="-106.68" y2="99.06" width="0.1524" layer="91"/>
+</segment>
+<segment>
+<pinref part="GND23" gate="1" pin="GND"/>
+<pinref part="C9" gate="G$1" pin="-"/>
+<wire x1="-121.92" y1="96.52" x2="-121.92" y2="104.14" width="0.1524" layer="91"/>
+</segment>
+<segment>
+<pinref part="GND24" gate="1" pin="GND"/>
+<pinref part="C8" gate="G$1" pin="-"/>
+<wire x1="-48.26" y1="96.52" x2="-48.26" y2="104.14" width="0.1524" layer="91"/>
 </segment>
 </net>
@@
 <wire x1="203.2" y1="63.5" x2="203.2" y2="60.96" width="0.1524" layer="91"/>
 <pinref part="IC2" gate="G$1" pin="BAT"/>
-<wire x1="187.96" y1="63.5" x2="195.58" y2="63.5" width="0.1524" layer="91"/>
+<wire x1="190.5" y1="63.5" x2="195.58" y2="63.5" width="0.1524" layer="91"/>
 <junction x="203.2" y="63.5"/>
 <wire x1="195.58" y1="63.5" x2="203.2" y2="63.5" width="0.1524" layer="91"/>
@@
 <pinref part="IC2" gate="G$1" pin="CE"/>
 <pinref part="R7" gate="G$1" pin="2"/>
-<wire x1="182.88" y1="81.28" x2="190.5" y2="81.28" width="0.1524" layer="91"/>
-<wire x1="190.5" y1="81.28" x2="190.5" y2="76.2" width="0.1524" layer="91"/>
-<wire x1="190.5" y1="76.2" x2="190.5" y2="71.12" width="0.1524" layer="91"/>
-<wire x1="190.5" y1="71.12" x2="187.96" y2="71.12" width="0.1524" layer="91"/>
+<wire x1="182.88" y1="81.28" x2="193.04" y2="81.28" width="0.1524" layer="91"/>
+<wire x1="193.04" y1="81.28" x2="193.04" y2="71.12" width="0.1524" layer="91"/>
+<wire x1="193.04" y1="71.12" x2="190.5" y2="71.12" width="0.1524" layer="91"/>
+<wire x1="190.5" y1="71.12" x2="190.5" y2="71.12" width="0.1524" layer="91"/>
 <pinref part="LED1" gate="G$1" pin="A"/>
-<wire x1="203.2" y1="78.74" x2="203.2" y2="81.28" width="0.1524" layer="91"/>
-<wire x1="203.2" y1="81.28" x2="190.5" y2="81.28" width="0.1524" layer="91"/>
-<junction x="190.5" y="81.28"/>
+<wire x1="205.74" y1="78.74" x2="205.74" y2="81.28" width="0.1524" layer="91"/>
+<wire x1="205.74" y1="81.28" x2="193.04" y2="81.28" width="0.1524" layer="91"/>
+<junction x="193.04" y="81.28"/>
 </segment>
 </net>
@@
 <pinref part="R21" gate="G$1" pin="2"/>
 <pinref part="LED1" gate="G$1" pin="C"/>
-<wire x1="200.66" y1="68.58" x2="203.2" y2="68.58" width="0.1524" layer="91"/>
-<wire x1="203.2" y1="68.58" x2="203.2" y2="71.12" width="0.1524" layer="91"/>
+<wire x1="203.2" y1="68.58" x2="205.74" y2="68.58" width="0.1524" layer="91"/>
+<wire x1="205.74" y1="68.58" x2="205.74" y2="71.12" width="0.1524" layer="91"/>
 </segment>
 </net>
@@
 <pinref part="R21" gate="G$1" pin="1"/>
 <pinref part="IC2" gate="G$1" pin="CHRG"/>
-<wire x1="190.5" y1="68.58" x2="187.96" y2="68.58" width="0.1524" layer="91"/>
+<wire x1="193.04" y1="68.58" x2="190.5" y2="68.58" width="0.1524" layer="91"/>
 </segment>
 </net>
@@
 </segment>
 </net>
+<net name="N$3" class="0">
+<segment>
+<pinref part="L1" gate="G$1" pin="2"/>
+<pinref part="D5" gate="G$1" pin="A"/>
+<wire x1="-76.2" y1="129.54" x2="-71.12" y2="129.54" width="0.1524" layer="91"/>
+<pinref part="T12" gate="A" pin="D"/>
+<wire x1="-71.12" y1="129.54" x2="-66.04" y2="129.54" width="0.1524" layer="91"/>
+<wire x1="-71.12" y1="121.92" x2="-71.12" y2="129.54" width="0.1524" layer="91"/>
+<junction x="-71.12" y="129.54"/>
+</segment>
+</net>
+<net name="N$15" class="0">
+<segment>
+<pinref part="T12" gate="A" pin="G"/>
+<pinref part="IC4" gate="G1" pin="EXT"/>
+<wire x1="-76.2" y1="114.3" x2="-78.74" y2="114.3" width="0.1524" layer="91"/>
+</segment>
+</net>
+<net name="N$24" class="0">
+<segment>
+<pinref part="L1" gate="G$1" pin="1"/>
+<wire x1="-104.14" y1="129.54" x2="-101.6" y2="129.54" width="0.1524" layer="91"/>
+<wire x1="-101.6" y1="129.54" x2="-86.36" y2="129.54" width="0.1524" layer="91"/>
+<wire x1="-104.14" y1="129.54" x2="-114.3" y2="129.54" width="0.1524" layer="91"/>
+<pinref part="C9" gate="G$1" pin="+"/>
+<wire x1="-121.92" y1="111.76" x2="-121.92" y2="129.54" width="0.1524" layer="91"/>
+<wire x1="-121.92" y1="129.54" x2="-114.3" y2="129.54" width="0.1524" layer="91"/>
+<wire x1="-121.92" y1="129.54" x2="-127" y2="129.54" width="0.1524" layer="91"/>
+<junction x="-121.92" y="129.54"/>
+<pinref part="R25" gate="G$1" pin="2"/>
+<wire x1="-101.6" y1="127" x2="-101.6" y2="129.54" width="0.1524" layer="91"/>
+<junction x="-101.6" y="129.54"/>
+</segment>
+</net>
+<net name="N$34" class="0">
+<segment>
+<pinref part="IC4" gate="G1" pin="OUT"/>
+<wire x1="-99.06" y1="109.22" x2="-106.68" y2="109.22" width="0.1524" layer="91"/>
+<wire x1="-106.68" y1="109.22" x2="-106.68" y2="139.7" width="0.1524" layer="91"/>
+<wire x1="-106.68" y1="139.7" x2="-58.42" y2="139.7" width="0.1524" layer="91"/>
+<wire x1="-58.42" y1="139.7" x2="-58.42" y2="129.54" width="0.1524" layer="91"/>
+<pinref part="D5" gate="G$1" pin="C"/>
+<wire x1="-58.42" y1="129.54" x2="-60.96" y2="129.54" width="0.1524" layer="91"/>
+<pinref part="C7" gate="G$1" pin="2"/>
+<wire x1="-106.68" y1="106.68" x2="-106.68" y2="109.22" width="0.1524" layer="91"/>
+<junction x="-106.68" y="109.22"/>
+<wire x1="-58.42" y1="129.54" x2="-53.34" y2="129.54" width="0.1524" layer="91"/>
+<junction x="-58.42" y="129.54"/>
+<pinref part="C8" gate="G$1" pin="+"/>
+<wire x1="-48.26" y1="111.76" x2="-48.26" y2="129.54" width="0.1524" layer="91"/>
+<wire x1="-48.26" y1="129.54" x2="-53.34" y2="129.54" width="0.1524" layer="91"/>
+<wire x1="-48.26" y1="129.54" x2="-43.18" y2="129.54" width="0.1524" layer="91"/>
+<junction x="-48.26" y="129.54"/>
+</segment>
+</net>
+<net name="N$18" class="0">
+<segment>
+<pinref part="IC4" gate="G1" pin="CE"/>
+<wire x1="-99.06" y1="114.3" x2="-101.6" y2="114.3" width="0.1524" layer="91"/>
+<pinref part="R25" gate="G$1" pin="1"/>
+<wire x1="-101.6" y1="114.3" x2="-101.6" y2="116.84" width="0.1524" layer="91"/>
+</segment>
+</net>

Commit message: pcb
Parts:
- added R26, R27, R28: 0, skydrop:R_1206
Connections:
- new net N$35: R26.2, R27.1
- new net N$36: MOTOR_A.P, R27.2
- new net N$37: R28.2, T4.D
- net BAT_CHECK: now also U1.GPIO14; no longer U1.GPIO12
- net H_BCK: now also U1.GPIO12; no longer U1.GPIO13
- net H_FWD: now also U1.GPIO13; no longer U1.GPIO14
- net N$33: now also R26.1; no longer MOTOR_A.P
- net N$4: now also R28.1; no longer T4.D
Other:
- moved on the sheet: MOTOR_A, MOTOR_B
Changed lines of the file:
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@@
 <part name="GND24" library="supply1" library_urn="urn:adsk.eagle:library:371" deviceset="GND" device=""/>
 <part name="R25" library="skydrop" deviceset="R_" device="1206" value="0"/>
+<part name="R26" library="skydrop" deviceset="R_" device="1206" value="0"/>
+<part name="R27" library="skydrop" deviceset="R_" device="1206" value="0"/>
+<part name="R28" library="skydrop" deviceset="R_" device="1206" value="0"/>
 </parts>
 <sheets>
@@
 <instance part="GND" gate="G$1" x="154.94" y="134.62" rot="MR0"/>
 <instance part="GND4" gate="1" x="149.86" y="124.46" rot="MR0"/>
-<instance part="MOTOR_B" gate="G$1" x="35.56" y="33.02"/>
-<instance part="MOTOR_A" gate="G$1" x="20.32" y="45.72" rot="R180"/>
+<instance part="MOTOR_B" gate="G$1" x="45.72" y="33.02"/>
+<instance part="MOTOR_A" gate="G$1" x="33.02" y="33.02" rot="R180"/>
 <instance part="BAT+" gate="G$1" x="259.08" y="63.5" rot="R180"/>
 <instance part="BAT-" gate="G$1" x="259.08" y="53.34" rot="R180"/>
@@
 <instance part="GND24" gate="1" x="-48.26" y="93.98"/>
 <instance part="R25" gate="G$1" x="-101.6" y="121.92" rot="R90"/>
+<instance part="R26" gate="G$1" x="10.16" y="33.02"/>
+<instance part="R27" gate="G$1" x="22.86" y="33.02"/>
+<instance part="R28" gate="G$1" x="53.34" y="40.64" rot="R90"/>
 </instances>
 <busses>
@@
 <wire x1="53.34" y1="33.02" x2="53.34" y2="30.48" width="0.1524" layer="91"/>
 <wire x1="50.8" y1="33.02" x2="53.34" y2="33.02" width="0.1524" layer="91"/>
+<pinref part="MOTOR_B" gate="G$1" pin="P"/>
+<wire x1="50.8" y1="33.02" x2="48.26" y2="33.02" width="0.1524" layer="91"/>
+<pinref part="R28" gate="G$1" pin="1"/>
 <wire x1="53.34" y1="35.56" x2="53.34" y2="33.02" width="0.1524" layer="91"/>
 <junction x="53.34" y="33.02"/>
-<pinref part="MOTOR_B" gate="G$1" pin="P"/>
-<wire x1="40.64" y1="33.02" x2="38.1" y2="33.02" width="0.1524" layer="91"/>
-<wire x1="50.8" y1="33.02" x2="40.64" y2="33.02" width="0.1524" layer="91"/>
-<pinref part="T4" gate="A" pin="D"/>
-<wire x1="53.34" y1="45.72" x2="53.34" y2="48.26" width="0.1524" layer="91"/>
-<wire x1="53.34" y1="35.56" x2="53.34" y2="45.72" width="0.1524" layer="91"/>
 </segment>
 </net>
@@
 <net name="H_BCK" class="0">
 <segment>
+<pinref part="R3" gate="G$1" pin="1"/>
+<wire x1="104.14" y1="33.02" x2="109.22" y2="33.02" width="0.1524" layer="91"/>
+<label x="111.76" y="33.02" size="1.778" layer="95"/>
+</segment>
+<segment>
+<pinref part="U1" gate="G$1" pin="GPIO12"/>
+<wire x1="60.96" y1="127" x2="43.18" y2="127" width="0.1524" layer="91"/>
+<label x="33.02" y="127" size="1.778" layer="95"/>
+</segment>
+</net>
+<net name="H_FWD" class="0">
+<segment>
+<pinref part="R4" gate="G$1" pin="2"/>
+<wire x1="-48.26" y1="33.02" x2="-53.34" y2="33.02" width="0.1524" layer="91"/>
+<label x="-63.5" y="33.02" size="1.778" layer="95"/>
+</segment>
+<segment>
 <pinref part="U1" gate="G$1" pin="GPIO13"/>
 <wire x1="60.96" y1="124.46" x2="43.18" y2="124.46" width="0.1524" layer="91"/>
 <label x="33.02" y="124.46" size="1.778" layer="95"/>
 </segment>
-<segment>
-<pinref part="R3" gate="G$1" pin="1"/>
-<wire x1="104.14" y1="33.02" x2="109.22" y2="33.02" width="0.1524" layer="91"/>
-<label x="111.76" y="33.02" size="1.778" layer="95"/>
-</segment>
-</net>
-<net name="H_FWD" class="0">
-<segment>
-<pinref part="U1" gate="G$1" pin="GPIO14"/>
-<wire x1="60.96" y1="129.54" x2="43.18" y2="129.54" width="0.1524" layer="91"/>
-<label x="33.02" y="129.54" size="1.778" layer="95"/>
-</segment>
-<segment>
-<pinref part="R4" gate="G$1" pin="2"/>
-<wire x1="-48.26" y1="33.02" x2="-53.34" y2="33.02" width="0.1524" layer="91"/>
-<label x="-63.5" y="33.02" size="1.778" layer="95"/>
-</segment>
 </net>
 <net name="H_PWM" class="0">
@@
 <net name="BAT_CHECK" class="0">
 <segment>
-<pinref part="U1" gate="G$1" pin="GPIO12"/>
-<wire x1="60.96" y1="127" x2="43.18" y2="127" width="0.1524" layer="91"/>
-<label x="27.94" y="127" size="1.778" layer="95"/>
-</segment>
-<segment>
 <pinref part="R14" gate="G$1" pin="2"/>
 <wire x1="137.16" y1="25.4" x2="137.16" y2="27.94" width="0.1524" layer="91"/>
 <label x="119.38" y="25.4" size="1.778" layer="95"/>
+</segment>
+<segment>
+<pinref part="U1" gate="G$1" pin="GPIO14"/>
+<wire x1="60.96" y1="129.54" x2="43.18" y2="129.54" width="0.1524" layer="91"/>
+<label x="27.94" y="129.54" size="1.778" layer="95"/>
 </segment>
 </net>
@@
 <net name="N$33" class="0">
 <segment>
-<pinref part="MOTOR_A" gate="G$1" pin="P"/>
-<wire x1="15.24" y1="45.72" x2="17.78" y2="45.72" width="0.1524" layer="91"/>
 <pinref part="T3" gate="A" pin="D"/>
 <wire x1="2.54" y1="43.18" x2="2.54" y2="45.72" width="0.1524" layer="91"/>
 <wire x1="2.54" y1="45.72" x2="2.54" y2="48.26" width="0.1524" layer="91"/>
-<wire x1="5.08" y1="45.72" x2="2.54" y2="45.72" width="0.1524" layer="91"/>
-<junction x="2.54" y="45.72"/>
 <pinref part="T1" gate="A" pin="D"/>
 <wire x1="2.54" y1="33.02" x2="2.54" y2="30.48" width="0.1524" layer="91"/>
 <wire x1="2.54" y1="43.18" x2="2.54" y2="33.02" width="0.1524" layer="91"/>
-<wire x1="15.24" y1="45.72" x2="5.08" y2="45.72" width="0.1524" layer="91"/>
+<pinref part="R26" gate="G$1" pin="1"/>
+<wire x1="5.08" y1="33.02" x2="2.54" y2="33.02" width="0.1524" layer="91"/>
+<junction x="2.54" y="33.02"/>
 </segment>
 </net>
@@
 </segment>
 </net>
+<net name="N$35" class="0">
+<segment>
+<pinref part="R27" gate="G$1" pin="1"/>
+<pinref part="R26" gate="G$1" pin="2"/>
+<wire x1="17.78" y1="33.02" x2="15.24" y2="33.02" width="0.1524" layer="91"/>
+</segment>
+</net>
+<net name="N$36" class="0">
+<segment>
+<pinref part="MOTOR_A" gate="G$1" pin="P"/>
+<pinref part="R27" gate="G$1" pin="2"/>
+<wire x1="30.48" y1="33.02" x2="27.94" y2="33.02" width="0.1524" layer="91"/>
+</segment>
+</net>
+<net name="N$37" class="0">
+<segment>
+<pinref part="T4" gate="A" pin="D"/>
+<pinref part="R28" gate="G$1" pin="2"/>
+<wire x1="53.34" y1="48.26" x2="53.34" y2="45.72" width="0.1524" layer="91"/>
+</segment>
+</net>
