File: pcb/rc.sch (EAGLE design)
At the start: 79 parts, among them IC2 TP4056

Commit message: pcb
Parts:
- added R29: 0, skydrop:R_1206
- U1: device esp8266modules:ESP12ESMD -> my:ESP-12
Connections:
- removed net N$34: C7.2, C8.+, D5.C, IC4.OUT
- new net 5V: C7.2, C8.+, D5.C, IC4.OUT, R23.2, R29.2
- net BAT_CHECK: now also U1.GPIO13; no longer U1.GPIO14
- net BAT_PROT: now also C9.+, L1.1, R25.2; no longer C6.1, IC3.EN, IC3.IN, R23.2
- net H_BCK: now also U1.GPIO14; no longer U1.GPIO12
- net H_FWD: now also U1.GPIO12; no longer U1.GPIO13
- net N$24: now also C6.1, IC3.EN, IC3.IN, R29.1; no longer C9.+, L1.1, R25.2
Changed lines of the file:
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@@
 <part name="SERVO_POWER" library="wirepad" library_urn="urn:adsk.eagle:library:412" deviceset="WIREPAD" device="SMD5-1,8" package3d_urn="urn:adsk.eagle:package:30844/1"/>
 <part name="SERVO_GND" library="wirepad" library_urn="urn:adsk.eagle:library:412" deviceset="WIREPAD" device="SMD5-1,8" package3d_urn="urn:adsk.eagle:package:30844/1"/>
-<part name="U1" library="esp8266modules" deviceset="ESP12E" device="SMD"/>
+<part name="U1" library="my" deviceset="ESP-12" device=""/>
 <part name="R15" library="skydrop" deviceset="R_" device="0805"/>
 <part name="R16" library="skydrop" deviceset="R_" device="0805"/>
@@
 <part name="R27" library="skydrop" deviceset="R_" device="1206" value="0"/>
 <part name="R28" library="skydrop" deviceset="R_" device="1206" value="0"/>
+<part name="R29" library="skydrop" deviceset="R_" device="1206" value="0"/>
 </parts>
 <sheets>
@@
 <instance part="SERVO_POWER" gate="G$1" x="248.92" y="160.02" rot="R180"/>
 <instance part="SERVO_GND" gate="G$1" x="248.92" y="152.4" rot="R180"/>
-<instance part="U1" gate="G$1" x="78.74" y="132.08"/>
+<instance part="U1" gate="G$1" x="78.74" y="134.62"/>
 <instance part="R15" gate="G$1" x="43.18" y="147.32" rot="R90"/>
 <instance part="R16" gate="G$1" x="33.02" y="147.32" rot="R90"/>
@@
 <instance part="R27" gate="G$1" x="22.86" y="33.02"/>
 <instance part="R28" gate="G$1" x="53.34" y="40.64" rot="R90"/>
+<instance part="R29" gate="G$1" x="-20.32" y="121.92" rot="R180"/>
 </instances>
 <busses>
@@
 <wire x1="165.1" y1="15.24" x2="165.1" y2="33.02" width="0.1524" layer="91"/>
 <junction x="165.1" y="33.02"/>
-</segment>
-<segment>
-<pinref part="IC3" gate="G1" pin="EN"/>
-<wire x1="2.54" y1="116.84" x2="0" y2="116.84" width="0.1524" layer="91"/>
-<wire x1="0" y1="116.84" x2="0" y2="121.92" width="0.1524" layer="91"/>
-<pinref part="IC3" gate="G1" pin="IN"/>
-<wire x1="0" y1="121.92" x2="2.54" y2="121.92" width="0.1524" layer="91"/>
-<pinref part="C6" gate="G$1" pin="1"/>
-<wire x1="-12.7" y1="114.3" x2="-12.7" y2="121.92" width="0.1524" layer="91"/>
-<wire x1="-12.7" y1="121.92" x2="0" y2="121.92" width="0.1524" layer="91"/>
-<junction x="0" y="121.92"/>
-<wire x1="-12.7" y1="121.92" x2="-17.78" y2="121.92" width="0.1524" layer="91"/>
-<junction x="-12.7" y="121.92"/>
-<label x="-33.02" y="121.92" size="1.778" layer="95"/>
-</segment>
-<segment>
-<pinref part="R23" gate="G$1" pin="2"/>
-<wire x1="233.68" y1="160.02" x2="223.52" y2="160.02" width="0.1524" layer="91"/>
-<label x="208.28" y="160.02" size="1.778" layer="95"/>
 </segment>
 <segment>
@@
 <junction x="25.4" y="71.12"/>
 <wire x1="25.4" y1="73.66" x2="25.4" y2="83.82" width="0.1524" layer="91"/>
+</segment>
+<segment>
+<pinref part="L1" gate="G$1" pin="1"/>
+<wire x1="-104.14" y1="129.54" x2="-101.6" y2="129.54" width="0.1524" layer="91"/>
+<wire x1="-101.6" y1="129.54" x2="-86.36" y2="129.54" width="0.1524" layer="91"/>
+<wire x1="-104.14" y1="129.54" x2="-114.3" y2="129.54" width="0.1524" layer="91"/>
+<pinref part="C9" gate="G$1" pin="+"/>
+<wire x1="-121.92" y1="111.76" x2="-121.92" y2="129.54" width="0.1524" layer="91"/>
+<wire x1="-121.92" y1="129.54" x2="-114.3" y2="129.54" width="0.1524" layer="91"/>
+<wire x1="-121.92" y1="129.54" x2="-127" y2="129.54" width="0.1524" layer="91"/>
+<junction x="-121.92" y="129.54"/>
+<pinref part="R25" gate="G$1" pin="2"/>
+<wire x1="-101.6" y1="127" x2="-101.6" y2="129.54" width="0.1524" layer="91"/>
+<junction x="-101.6" y="129.54"/>
+<label x="-132.08" y="132.08" size="1.778" layer="95"/>
 </segment>
 </net>
@@
 </segment>
 <segment>
-<pinref part="U1" gate="G$1" pin="GPIO12"/>
-<wire x1="60.96" y1="127" x2="43.18" y2="127" width="0.1524" layer="91"/>
-<label x="33.02" y="127" size="1.778" layer="95"/>
+<pinref part="U1" gate="G$1" pin="GPIO14"/>
+<wire x1="60.96" y1="129.54" x2="40.64" y2="129.54" width="0.1524" layer="91"/>
+<label x="30.48" y="129.54" size="1.778" layer="95"/>
 </segment>
 </net>
@@
 </segment>
 <segment>
-<pinref part="U1" gate="G$1" pin="GPIO13"/>
-<wire x1="60.96" y1="124.46" x2="43.18" y2="124.46" width="0.1524" layer="91"/>
-<label x="33.02" y="124.46" size="1.778" layer="95"/>
+<pinref part="U1" gate="G$1" pin="GPIO12"/>
+<wire x1="60.96" y1="127" x2="40.64" y2="127" width="0.1524" layer="91"/>
+<label x="30.48" y="127" size="1.778" layer="95"/>
 </segment>
 </net>
@@
 </segment>
 <segment>
-<pinref part="U1" gate="G$1" pin="GPIO14"/>
-<wire x1="60.96" y1="129.54" x2="43.18" y2="129.54" width="0.1524" layer="91"/>
-<label x="27.94" y="129.54" size="1.778" layer="95"/>
+<pinref part="U1" gate="G$1" pin="GPIO13"/>
+<wire x1="60.96" y1="124.46" x2="40.64" y2="124.46" width="0.1524" layer="91"/>
+<label x="25.4" y="124.46" size="1.778" layer="95"/>
 </segment>
 </net>
@@
 </segment>
 </net>
-<net name="N$24" class="0">
-<segment>
-<pinref part="L1" gate="G$1" pin="1"/>
-<wire x1="-104.14" y1="129.54" x2="-101.6" y2="129.54" width="0.1524" layer="91"/>
-<wire x1="-101.6" y1="129.54" x2="-86.36" y2="129.54" width="0.1524" layer="91"/>
-<wire x1="-104.14" y1="129.54" x2="-114.3" y2="129.54" width="0.1524" layer="91"/>
-<pinref part="C9" gate="G$1" pin="+"/>
-<wire x1="-121.92" y1="111.76" x2="-121.92" y2="129.54" width="0.1524" layer="91"/>
-<wire x1="-121.92" y1="129.54" x2="-114.3" y2="129.54" width="0.1524" layer="91"/>
-<wire x1="-121.92" y1="129.54" x2="-127" y2="129.54" width="0.1524" layer="91"/>
-<junction x="-121.92" y="129.54"/>
-<pinref part="R25" gate="G$1" pin="2"/>
-<wire x1="-101.6" y1="127" x2="-101.6" y2="129.54" width="0.1524" layer="91"/>
-<junction x="-101.6" y="129.54"/>
-</segment>
-</net>
-<net name="N$34" class="0">
+<net name="N$18" class="0">
+<segment>
+<pinref part="IC4" gate="G1" pin="CE"/>
+<wire x1="-99.06" y1="114.3" x2="-101.6" y2="114.3" width="0.1524" layer="91"/>
+<pinref part="R25" gate="G$1" pin="1"/>
+<wire x1="-101.6" y1="114.3" x2="-101.6" y2="116.84" width="0.1524" layer="91"/>
+</segment>
+</net>
+<net name="N$35" class="0">
+<segment>
+<pinref part="R27" gate="G$1" pin="1"/>
+<pinref part="R26" gate="G$1" pin="2"/>
+<wire x1="17.78" y1="33.02" x2="15.24" y2="33.02" width="0.1524" layer="91"/>
+</segment>
+</net>
+<net name="N$36" class="0">
+<segment>
+<pinref part="MOTOR_A" gate="G$1" pin="P"/>
+<pinref part="R27" gate="G$1" pin="2"/>
+<wire x1="30.48" y1="33.02" x2="27.94" y2="33.02" width="0.1524" layer="91"/>
+</segment>
+</net>
+<net name="N$37" class="0">
+<segment>
+<pinref part="T4" gate="A" pin="D"/>
+<pinref part="R28" gate="G$1" pin="2"/>
+<wire x1="53.34" y1="48.26" x2="53.34" y2="45.72" width="0.1524" layer="91"/>
+</segment>
+</net>
+<net name="5V" class="0">
 <segment>
 <pinref part="IC4" gate="G1" pin="OUT"/>
@@
 <wire x1="-48.26" y1="129.54" x2="-43.18" y2="129.54" width="0.1524" layer="91"/>
 <junction x="-48.26" y="129.54"/>
-</segment>
-</net>
-<net name="N$18" class="0">
-<segment>
-<pinref part="IC4" gate="G1" pin="CE"/>
-<wire x1="-99.06" y1="114.3" x2="-101.6" y2="114.3" width="0.1524" layer="91"/>
-<pinref part="R25" gate="G$1" pin="1"/>
-<wire x1="-101.6" y1="114.3" x2="-101.6" y2="116.84" width="0.1524" layer="91"/>
-</segment>
-</net>
-<net name="N$35" class="0">
-<segment>
-<pinref part="R27" gate="G$1" pin="1"/>
-<pinref part="R26" gate="G$1" pin="2"/>
-<wire x1="17.78" y1="33.02" x2="15.24" y2="33.02" width="0.1524" layer="91"/>
-</segment>
-</net>
-<net name="N$36" class="0">
-<segment>
-<pinref part="MOTOR_A" gate="G$1" pin="P"/>
-<pinref part="R27" gate="G$1" pin="2"/>
-<wire x1="30.48" y1="33.02" x2="27.94" y2="33.02" width="0.1524" layer="91"/>
-</segment>
-</net>
-<net name="N$37" class="0">
-<segment>
-<pinref part="T4" gate="A" pin="D"/>
-<pinref part="R28" gate="G$1" pin="2"/>
-<wire x1="53.34" y1="48.26" x2="53.34" y2="45.72" width="0.1524" layer="91"/>
+<label x="-40.64" y="129.54" size="1.778" layer="95"/>
+</segment>
+<segment>
+<pinref part="R23" gate="G$1" pin="2"/>
+<wire x1="233.68" y1="160.02" x2="223.52" y2="160.02" width="0.1524" layer="91"/>
+<label x="218.44" y="160.02" size="1.778" layer="95"/>
+</segment>
+<segment>
+<pinref part="R29" gate="G$1" pin="2"/>
+<wire x1="-25.4" y1="121.92" x2="-27.94" y2="121.92" width="0.1524" layer="91"/>
+<label x="-30.48" y="124.46" size="1.778" layer="95"/>
+</segment>
+</net>
+<net name="N$24" class="0">
+<segment>
+<pinref part="IC3" gate="G1" pin="EN"/>
+<wire x1="2.54" y1="116.84" x2="0" y2="116.84" width="0.1524" layer="91"/>
+<wire x1="0" y1="116.84" x2="0" y2="121.92" width="0.1524" layer="91"/>
+<pinref part="IC3" gate="G1" pin="IN"/>
+<wire x1="0" y1="121.92" x2="2.54" y2="121.92" width="0.1524" layer="91"/>
+<pinref part="C6" gate="G$1" pin="1"/>
+<wire x1="-12.7" y1="114.3" x2="-12.7" y2="121.92" width="0.1524" layer="91"/>
+<wire x1="-12.7" y1="121.92" x2="0" y2="121.92" width="0.1524" layer="91"/>
+<junction x="0" y="121.92"/>
+<pinref part="R29" gate="G$1" pin="1"/>
+<wire x1="-15.24" y1="121.92" x2="-12.7" y2="121.92" width="0.1524" layer="91"/>
+<junction x="-12.7" y="121.92"/>
 </segment>
 </net>
@@
 </drawing>
 <compatibility>
-<note version="6.3" minversion="6.2.2" severity="warning">
-Since Version 6.2.2 text objects can contain more than one line,
-which will not be processed correctly with this version.
-</note>
 <note version="8.2" severity="warning">
 Since Version 8.2, EAGLE supports online libraries. The ids

Commit message: pcb
Parts:
- removed JP4: (no value), adafruit:PINHD-1X1
- removed JP5: (no value), adafruit:PINHD-1X3
- added JP6: (no value), pinhead:PINHD-1X2
- JP1, JP2: device adafruit:PINHD-1X3 -> pinhead:PINHD-1X3
- JP3: device adafruit:PINHD-1X1 -> pinhead:PINHD-1X3
Other:
- moved on the sheet: JP1, JP2
Changed lines of the file:
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@@
 <setting verticaltext="up"/>
 </settings>
-<grid distance="0.1" unitdist="inch" unit="inch" style="dots" multiple="1" display="yes" altdistance="0.01" altunitdist="inch" altunit="inch"/>
+<grid distance="0.1" unitdist="inch" unit="inch" style="lines" multiple="1" display="no" altdistance="0.01" altunitdist="inch" altunit="inch"/>
 <layers>
 <layer number="1" name="Top" color="4" fill="11" visible="no" active="no"/>
@@
 <part name="FLASH2" library="wirepad" library_urn="urn:adsk.eagle:library:412" deviceset="WIREPAD" device="SMD5-1,8" package3d_urn="urn:adsk.eagle:package:30844/1" value="WIREPADSMD5-1,8"/>
 <part name="GND21" library="supply1" library_urn="urn:adsk.eagle:library:371" deviceset="GND" device=""/>
-<part name="JP1" library="adafruit" deviceset="PINHD-1X3" device=""/>
-<part name="JP2" library="adafruit" deviceset="PINHD-1X3" device=""/>
-<part name="JP5" library="adafruit" deviceset="PINHD-1X3" device=""/>
-<part name="JP3" library="adafruit" deviceset="PINHD-1X1" device=""/>
-<part name="JP4" library="adafruit" deviceset="PINHD-1X1" device=""/>
 <part name="GND19" library="supply1" library_urn="urn:adsk.eagle:library:371" deviceset="GND" device=""/>
 <part name="IC4" library="my" deviceset="NCP1450A" device=""/>
@@
 <part name="R28" library="skydrop" deviceset="R_" device="1206" value="0"/>
 <part name="R29" library="skydrop" deviceset="R_" device="1206" value="0"/>
+<part name="JP6" library="pinhead" library_urn="urn:adsk.eagle:library:325" deviceset="PINHD-1X2" device="" package3d_urn="urn:adsk.eagle:package:22435/2"/>
+<part name="JP1" library="pinhead" library_urn="urn:adsk.eagle:library:325" deviceset="PINHD-1X3" device="" package3d_urn="urn:adsk.eagle:package:22458/2"/>
+<part name="JP2" library="pinhead" library_urn="urn:adsk.eagle:library:325" deviceset="PINHD-1X3" device="" package3d_urn="urn:adsk.eagle:package:22458/2"/>
+<part name="JP3" library="pinhead" library_urn="urn:adsk.eagle:library:325" deviceset="PINHD-1X3" device="" package3d_urn="urn:adsk.eagle:package:22458/2"/>
 </parts>
 <sheets>
@@
 <instance part="FLASH2" gate="G$1" x="129.54" y="127" rot="MR0"/>
 <instance part="GND21" gate="1" x="124.46" y="119.38" rot="MR0"/>
-<instance part="JP1" gate="A" x="165.1" y="137.16"/>
-<instance part="JP2" gate="A" x="266.7" y="160.02"/>
-<instance part="JP5" gate="A" x="195.58" y="137.16"/>
-<instance part="JP3" gate="G$1" x="167.64" y="119.38"/>
-<instance part="JP4" gate="G$1" x="167.64" y="114.3"/>
 <instance part="GND19" gate="1" x="175.26" y="53.34"/>
 <instance part="IC4" gate="G1" x="-88.9" y="109.22"/>
@@
 <instance part="R28" gate="G$1" x="53.34" y="40.64" rot="R90"/>
 <instance part="R29" gate="G$1" x="-20.32" y="121.92" rot="R180"/>
+<instance part="JP6" gate="G$1" x="142.24" y="119.38"/>
+<instance part="JP1" gate="A" x="167.64" y="137.16"/>
+<instance part="JP2" gate="A" x="264.16" y="160.02"/>
+<instance part="JP3" gate="A" x="264.16" y="124.46"/>
 </instances>
 <busses>
