File: pcb/rc.sch (EAGLE design)
At the start: 79 parts, among them IC2 TP4056

Commit message: pcb
Parts:
- removed FLASH1, FLASH2, GND, RX, SERVO_CONTROL, SERVO_GND, SERVO_POWER, TX: WIREPADSMD5-1,8, wirepad:WIREPADSMD5-1,8
- removed JP2, JP3: (no value), pinhead:PINHD-1X3
- added JP4, JP5: (no value), my:PINHD-1X3
- JP1: device pinhead:PINHD-1X3 -> my:PINHD-1X3
- JP6: device pinhead:PINHD-1X2 -> my:PINHD-1X2
Connections:
- net SERVO_CONTROL renamed SERVO#1_CTRL
- removed net N$29: R22.1, SERVO_CONTROL.P
- new net SERVO#2_CTRL: JP1.1, R18.1, U1.GPIO2
- net 5V: now also JP1.2
- net GND: now also JP1.3, JP4.3, JP5.3, JP6.2; no longer FLASH2.P, GND.P, SERVO_GND.P
- net N$21: now also JP6.1; no longer FLASH1.P
- net N$22: now also JP4.1, R22.1; no longer R18.1, U1.GPIO2
- net N$30: now also JP4.2; no longer SERVO_POWER.P
- net RX: now also JP5.2; no longer RX.P
- net TX: now also JP5.1; no longer TX.P
Other:
- moved on the sheet: JP1, JP6, R17, R18, R22, R23

Commit message: pcb
Parts:
- removed R14, R23, R26, R27: 0, skydrop:R_1206
Connections:
- removed net N$14 (its old number): R14.1, T11.C
- removed net N$24: C6.1, IC3.EN, IC3.IN, R29.1
- removed net N$30: JP4.2, R23.1
- removed net N$33: R26.1, T1.D, T3.D
- removed net N$35: R26.2, R27.1
- new net N$29: C7.2, C8.+, D5.C, IC4.OUT, R29.2
- net 5V: now also C6.1, IC3.EN, IC3.IN, JP4.2, R29.1; no longer C7.2, C8.+, D5.C, IC4.OUT, R23.2, R29.2
- net BAT_CHECK: now also T11.C; no longer R14.2
- net N$36: now also T1.D, T3.D; no longer R27.2
Other:
- moved on the sheet: JP1, MOTOR_B, R29

Commit message: pcb
Parts:
- removed D5: (no value), adafruit:DIODESMA
- added D1: (no value), semicon-smd-ipc:D-FILL-SMB
- C5, C6: device skydrop:C_1206 -> skydrop:C_0805
- C8, C9: device adafruit:CPOL-USD/7343-31W -> adafruit:CPOL-USCT6032
- L1: value (none) -> DR74; device inductor-neosid:MS85 -> inductors:DR74
- R2: device skydrop:R_0805 -> my:R_08050805
Connections:
- net N$29: now also D1.C; no longer D5.C
- net N$3: now also D1.A; no longer D5.A
Changed lines of the file:
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@@
 <setting verticaltext="up"/>
 </settings>
-<grid distance="0.1" unitdist="inch" unit="inch" style="dots" multiple="1" display="no" altdistance="0.01" altunitdist="inch" altunit="inch"/>
+<grid distance="0.1" unitdist="inch" unit="inch" style="lines" multiple="1" display="no" altdistance="0.01" altunitdist="inch" altunit="inch"/>
 <layers>
 <layer number="1" name="Top" color="4" fill="11" visible="no" active="no"/>
@@
 <part name="R10" library="skydrop" deviceset="R_" device="0805"/>
 <part name="R1" library="skydrop" deviceset="R_" device="0805"/>
-<part name="R2" library="skydrop" deviceset="R_" device="0805"/>
+<part name="R2" library="my" deviceset="R_0805" device="0805"/>
 <part name="R3" library="skydrop" deviceset="R_" device="0805"/>
 <part name="R4" library="skydrop" deviceset="R_" device="0805"/>
@@
 <part name="C4" library="skydrop" deviceset="C-EU" device="C0805"/>
 <part name="GND14" library="supply1" library_urn="urn:adsk.eagle:library:371" deviceset="GND" device=""/>
-<part name="C5" library="skydrop" deviceset="C_" device="1206"/>
-<part name="C6" library="skydrop" deviceset="C_" device="1206"/>
+<part name="C5" library="skydrop" deviceset="C_" device="0805"/>
+<part name="C6" library="skydrop" deviceset="C_" device="0805"/>
 <part name="GND15" library="supply1" library_urn="urn:adsk.eagle:library:371" deviceset="GND" device=""/>
 <part name="GND16" library="supply1" library_urn="urn:adsk.eagle:library:371" deviceset="GND" device=""/>
@@
 <part name="GND19" library="supply1" library_urn="urn:adsk.eagle:library:371" deviceset="GND" device=""/>
 <part name="IC4" library="my" deviceset="NCP1450A" device=""/>
-<part name="D5" library="adafruit" deviceset="DIODE" device="SMA"/>
-<part name="L1" library="inductor-neosid" library_urn="urn:adsk.eagle:library:241" deviceset="MS85" device="" package3d_urn="urn:adsk.eagle:package:14698/1"/>
+<part name="L1" library="inductors" library_urn="urn:adsk.eagle:library:243" deviceset="DR74" device="" package3d_urn="urn:adsk.eagle:package:15122/1"/>
 <part name="T12" library="zetex" library_urn="urn:adsk.eagle:library:418" deviceset="NMOSSOT23" device="" package3d_urn="urn:adsk.eagle:package:30981/1"/>
 <part name="GND20" library="supply1" library_urn="urn:adsk.eagle:library:371" deviceset="GND" device=""/>
 <part name="C7" library="skydrop" deviceset="C-EU" device="C0805"/>
 <part name="GND22" library="supply1" library_urn="urn:adsk.eagle:library:371" deviceset="GND" device=""/>
-<part name="C8" library="adafruit" deviceset="CPOL-US" device="D/7343-31W"/>
-<part name="C9" library="adafruit" deviceset="CPOL-US" device="D/7343-31W"/>
+<part name="C8" library="adafruit" deviceset="CPOL-US" device="CT6032"/>
+<part name="C9" library="adafruit" deviceset="CPOL-US" device="CT6032"/>
 <part name="GND23" library="supply1" library_urn="urn:adsk.eagle:library:371" deviceset="GND" device=""/>
 <part name="GND24" library="supply1" library_urn="urn:adsk.eagle:library:371" deviceset="GND" device=""/>
@@
 <part name="GND25" library="supply1" library_urn="urn:adsk.eagle:library:371" deviceset="GND" device=""/>
 <part name="R22" library="skydrop" deviceset="R_" device="1206" value="0"/>
+<part name="D1" library="semicon-smd-ipc" library_urn="urn:adsk.eagle:library:353" deviceset="D-FILL-" device="SMB" package3d_urn="urn:adsk.eagle:package:26311/1"/>
 </parts>
 <sheets>
@@
 <instance part="GND19" gate="1" x="175.26" y="53.34"/>
 <instance part="IC4" gate="G1" x="-88.9" y="109.22"/>
-<instance part="D5" gate="G$1" x="-63.5" y="129.54"/>
-<instance part="L1" gate="G$1" x="-81.28" y="129.54"/>
+<instance part="L1" gate="G$1" x="-86.36" y="129.54"/>
 <instance part="T12" gate="A" x="-71.12" y="116.84"/>
 <instance part="GND20" gate="1" x="-71.12" y="93.98"/>
@@
 <instance part="GND25" gate="1" x="241.3" y="139.7"/>
 <instance part="R22" gate="G$1" x="236.22" y="167.64" rot="R180"/>
+<instance part="D1" gate="G$1" x="-63.5" y="129.54"/>
 </instances>
 <busses>
@@
 <pinref part="L1" gate="G$1" pin="1"/>
 <wire x1="-104.14" y1="129.54" x2="-101.6" y2="129.54" width="0.1524" layer="91"/>
-<wire x1="-101.6" y1="129.54" x2="-86.36" y2="129.54" width="0.1524" layer="91"/>
+<wire x1="-101.6" y1="129.54" x2="-93.98" y2="129.54" width="0.1524" layer="91"/>
 <wire x1="-104.14" y1="129.54" x2="-114.3" y2="129.54" width="0.1524" layer="91"/>
 <pinref part="C9" gate="G$1" pin="+"/>
@@
 <segment>
 <pinref part="L1" gate="G$1" pin="2"/>
-<pinref part="D5" gate="G$1" pin="A"/>
-<wire x1="-76.2" y1="129.54" x2="-71.12" y2="129.54" width="0.1524" layer="91"/>
+<wire x1="-78.74" y1="129.54" x2="-71.12" y2="129.54" width="0.1524" layer="91"/>
 <pinref part="T12" gate="A" pin="D"/>
-<wire x1="-71.12" y1="129.54" x2="-66.04" y2="129.54" width="0.1524" layer="91"/>
 <wire x1="-71.12" y1="121.92" x2="-71.12" y2="129.54" width="0.1524" layer="91"/>
+<pinref part="D1" gate="G$1" pin="A"/>
+<wire x1="-66.04" y1="129.54" x2="-71.12" y2="129.54" width="0.1524" layer="91"/>
 <junction x="-71.12" y="129.54"/>
 </segment>
@@
 <wire x1="-106.68" y1="109.22" x2="-106.68" y2="137.16" width="0.1524" layer="91"/>
 <junction x="-106.68" y="109.22"/>
-<wire x1="-106.68" y1="137.16" x2="-58.42" y2="137.16" width="0.1524" layer="91"/>
-<wire x1="-58.42" y1="137.16" x2="-58.42" y2="129.54" width="0.1524" layer="91"/>
-<pinref part="D5" gate="G$1" pin="C"/>
-<wire x1="-58.42" y1="129.54" x2="-60.96" y2="129.54" width="0.1524" layer="91"/>
+<wire x1="-106.68" y1="137.16" x2="-55.88" y2="137.16" width="0.1524" layer="91"/>
+<wire x1="-55.88" y1="137.16" x2="-55.88" y2="129.54" width="0.1524" layer="91"/>
 <pinref part="C8" gate="G$1" pin="+"/>
 <wire x1="-48.26" y1="111.76" x2="-48.26" y2="129.54" width="0.1524" layer="91"/>
-<wire x1="-48.26" y1="129.54" x2="-58.42" y2="129.54" width="0.1524" layer="91"/>
-<junction x="-58.42" y="129.54"/>
+<wire x1="-48.26" y1="129.54" x2="-55.88" y2="129.54" width="0.1524" layer="91"/>
 <pinref part="R29" gate="G$1" pin="2"/>
 <wire x1="-45.72" y1="129.54" x2="-48.26" y2="129.54" width="0.1524" layer="91"/>
 <junction x="-48.26" y="129.54"/>
+<pinref part="D1" gate="G$1" pin="C"/>
+<wire x1="-60.96" y1="129.54" x2="-55.88" y2="129.54" width="0.1524" layer="91"/>
+<junction x="-55.88" y="129.54"/>
 </segment>
 </net>
@@
 packages will not be understood (or retained) with this version.
 </note>
+<note version="8.4" severity="warning">
+Since Version 8.4, EAGLE supports properties for SPICE simulation.
+Probes in schematics and SPICE mapping objects found in parts and library devices
+will not be understood with this version. Update EAGLE to the latest version
+for full support of SPICE simulation.
+</note>
 </compatibility>

Commit message: pcb
Parts:
- removed R22: 0, skydrop:R_1206
- added LED2: (no value), led:LEDCHIPLED_0805
Connections:
- removed net N$22: JP4.1, R22.1
- new net N$24: LED2.A, R17.1
- net H_PWM: now also R18.1, U1.GPIO2; no longer U1.GPIO5
- net N$21: now also LED2.C; no longer R17.1
- net SERVO#1_CTRL: now also JP1.1; no longer R22.2
- net SERVO#2_CTRL: now also JP4.1, U1.GPIO5; no longer JP1.1, R18.1, U1.GPIO2
Other:
- moved on the sheet: R15, R16, R17, R18
Changed lines of the file:
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@@
 <part name="JP1" library="my" deviceset="PINHD-1X3" device=""/>
 <part name="GND25" library="supply1" library_urn="urn:adsk.eagle:library:371" deviceset="GND" device=""/>
-<part name="R22" library="skydrop" deviceset="R_" device="1206" value="0"/>
 <part name="D1" library="semicon-smd-ipc" library_urn="urn:adsk.eagle:library:353" deviceset="D-FILL-" device="SMB" package3d_urn="urn:adsk.eagle:package:26311/1"/>
+<part name="LED2" library="led" library_urn="urn:adsk.eagle:library:259" deviceset="LED" device="CHIPLED_0805" package3d_urn="urn:adsk.eagle:package:15821/2"/>
 </parts>
 <sheets>
@@
 <instance part="GND5" gate="1" x="241.3" y="33.02"/>
 <instance part="U1" gate="G$1" x="78.74" y="134.62"/>
-<instance part="R15" gate="G$1" x="43.18" y="147.32" rot="R90"/>
-<instance part="R16" gate="G$1" x="33.02" y="147.32" rot="R90"/>
-<instance part="R17" gate="G$1" x="101.6" y="147.32" rot="R90"/>
-<instance part="R18" gate="G$1" x="106.68" y="147.32" rot="R90"/>
-<instance part="P+3" gate="VCC" x="58.42" y="167.64"/>
+<instance part="R15" gate="G$1" x="43.18" y="157.48" rot="R90"/>
+<instance part="R16" gate="G$1" x="33.02" y="157.48" rot="R90"/>
+<instance part="R17" gate="G$1" x="101.6" y="157.48" rot="R90"/>
+<instance part="R18" gate="G$1" x="106.68" y="157.48" rot="R90"/>
+<instance part="P+3" gate="VCC" x="58.42" y="177.8"/>
 <instance part="GND7" gate="1" x="96.52" y="101.6"/>
 <instance part="R19" gate="G$1" x="106.68" y="116.84" rot="R90"/>
@@
 <instance part="JP1" gate="A" x="251.46" y="149.86"/>
 <instance part="GND25" gate="1" x="241.3" y="139.7"/>
-<instance part="R22" gate="G$1" x="236.22" y="167.64" rot="R180"/>
 <instance part="D1" gate="G$1" x="-63.5" y="129.54"/>
+<instance part="LED2" gate="G$1" x="101.6" y="147.32"/>
 </instances>
 <busses>
@@
 <wire x1="60.96" y1="121.92" x2="58.42" y2="121.92" width="0.1524" layer="91"/>
 <pinref part="P+3" gate="VCC" pin="VCC"/>
-<wire x1="58.42" y1="121.92" x2="58.42" y2="157.48" width="0.1524" layer="91"/>
+<wire x1="58.42" y1="121.92" x2="58.42" y2="167.64" width="0.1524" layer="91"/>
 <pinref part="R15" gate="G$1" pin="2"/>
-<wire x1="58.42" y1="157.48" x2="58.42" y2="165.1" width="0.1524" layer="91"/>
-<wire x1="43.18" y1="152.4" x2="43.18" y2="157.48" width="0.1524" layer="91"/>
-<wire x1="43.18" y1="157.48" x2="58.42" y2="157.48" width="0.1524" layer="91"/>
+<wire x1="58.42" y1="167.64" x2="58.42" y2="175.26" width="0.1524" layer="91"/>
+<wire x1="43.18" y1="162.56" x2="43.18" y2="167.64" width="0.1524" layer="91"/>
+<wire x1="43.18" y1="167.64" x2="58.42" y2="167.64" width="0.1524" layer="91"/>
 <pinref part="R17" gate="G$1" pin="2"/>
-<wire x1="58.42" y1="157.48" x2="101.6" y2="157.48" width="0.1524" layer="91"/>
-<wire x1="101.6" y1="157.48" x2="101.6" y2="152.4" width="0.1524" layer="91"/>
+<wire x1="58.42" y1="167.64" x2="101.6" y2="167.64" width="0.1524" layer="91"/>
+<wire x1="101.6" y1="167.64" x2="101.6" y2="162.56" width="0.1524" layer="91"/>
 <pinref part="R18" gate="G$1" pin="2"/>
-<wire x1="106.68" y1="152.4" x2="106.68" y2="157.48" width="0.1524" layer="91"/>
-<wire x1="106.68" y1="157.48" x2="101.6" y2="157.48" width="0.1524" layer="91"/>
-<junction x="101.6" y="157.48"/>
+<wire x1="106.68" y1="162.56" x2="106.68" y2="167.64" width="0.1524" layer="91"/>
+<wire x1="106.68" y1="167.64" x2="101.6" y2="167.64" width="0.1524" layer="91"/>
+<junction x="101.6" y="167.64"/>
 <pinref part="R16" gate="G$1" pin="2"/>
-<wire x1="33.02" y1="152.4" x2="33.02" y2="157.48" width="0.1524" layer="91"/>
-<wire x1="33.02" y1="157.48" x2="43.18" y2="157.48" width="0.1524" layer="91"/>
-<junction x="43.18" y="157.48"/>
-<junction x="58.42" y="157.48"/>
+<wire x1="33.02" y1="162.56" x2="33.02" y2="167.64" width="0.1524" layer="91"/>
+<wire x1="33.02" y1="167.64" x2="43.18" y2="167.64" width="0.1524" layer="91"/>
+<junction x="43.18" y="167.64"/>
+<junction x="58.42" y="167.64"/>
 <pinref part="C1" gate="G$1" pin="2"/>
 <wire x1="58.42" y1="119.38" x2="58.42" y2="121.92" width="0.1524" layer="91"/>
@@
 <pinref part="R15" gate="G$1" pin="1"/>
 <wire x1="60.96" y1="139.7" x2="43.18" y2="139.7" width="0.1524" layer="91"/>
-<wire x1="43.18" y1="139.7" x2="43.18" y2="142.24" width="0.1524" layer="91"/>
+<wire x1="43.18" y1="139.7" x2="43.18" y2="152.4" width="0.1524" layer="91"/>
 <pinref part="R20" gate="G$1" pin="2"/>
 <wire x1="45.72" y1="132.08" x2="43.18" y2="132.08" width="0.1524" layer="91"/>
@@
 <pinref part="R16" gate="G$1" pin="1"/>
 <wire x1="60.96" y1="134.62" x2="33.02" y2="134.62" width="0.1524" layer="91"/>
-<wire x1="33.02" y1="134.62" x2="33.02" y2="142.24" width="0.1524" layer="91"/>
+<wire x1="33.02" y1="134.62" x2="33.02" y2="152.4" width="0.1524" layer="91"/>
 </segment>
 </net>
 <net name="N$21" class="0">
 <segment>
-<pinref part="R17" gate="G$1" pin="1"/>
-<wire x1="101.6" y1="142.24" x2="101.6" y2="129.54" width="0.1524" layer="91"/>
 <pinref part="U1" gate="G$1" pin="GPIO0"/>
 <wire x1="101.6" y1="129.54" x2="93.98" y2="129.54" width="0.1524" layer="91"/>
-<junction x="101.6" y="129.54"/>
 <pinref part="JP6" gate="G$1" pin="1"/>
 <wire x1="121.92" y1="111.76" x2="116.84" y2="111.76" width="0.1524" layer="91"/>
@@
 <wire x1="114.3" y1="129.54" x2="114.3" y2="111.76" width="0.1524" layer="91"/>
 <wire x1="114.3" y1="111.76" x2="116.84" y2="111.76" width="0.1524" layer="91"/>
+<pinref part="LED2" gate="G$1" pin="C"/>
+<wire x1="101.6" y1="142.24" x2="101.6" y2="129.54" width="0.1524" layer="91"/>
+<junction x="101.6" y="129.54"/>
 </segment>
 </net>
 <net name="SERVO#2_CTRL" class="0">
 <segment>
-<pinref part="U1" gate="G$1" pin="GPIO2"/>
-<wire x1="93.98" y1="127" x2="106.68" y2="127" width="0.1524" layer="91"/>
-<pinref part="R18" gate="G$1" pin="1"/>
-<wire x1="106.68" y1="127" x2="106.68" y2="142.24" width="0.1524" layer="91"/>
-<wire x1="106.68" y1="127" x2="119.38" y2="127" width="0.1524" layer="91"/>
-<junction x="106.68" y="127"/>
-<label x="121.92" y="127" size="1.778" layer="95"/>
-</segment>
-<segment>
-<pinref part="JP1" gate="A" pin="1"/>
-<wire x1="248.92" y1="152.4" x2="218.44" y2="152.4" width="0.1524" layer="91"/>
-<label x="193.04" y="152.4" size="1.778" layer="95"/>
+<pinref part="U1" gate="G$1" pin="GPIO5"/>
+<wire x1="93.98" y1="134.62" x2="119.38" y2="134.62" width="0.1524" layer="91"/>
+<label x="121.92" y="134.62" size="1.778" layer="95"/>
+</segment>
+<segment>
+<pinref part="JP4" gate="A" pin="1"/>
+<wire x1="248.92" y1="167.64" x2="218.44" y2="167.64" width="0.1524" layer="91"/>
+<label x="198.12" y="167.64" size="1.778" layer="95"/>
 </segment>
 </net>
@@
 <net name="H_PWM" class="0">
 <segment>
-<pinref part="U1" gate="G$1" pin="GPIO5"/>
-<wire x1="93.98" y1="134.62" x2="119.38" y2="134.62" width="0.1524" layer="91"/>
-<label x="121.92" y="134.62" size="1.778" layer="95"/>
-</segment>
-<segment>
 <pinref part="R5" gate="G$1" pin="2"/>
 <wire x1="-48.26" y1="-27.94" x2="-55.88" y2="-27.94" width="0.1524" layer="91"/>
 <label x="-60.96" y="-22.86" size="1.778" layer="95"/>
+</segment>
+<segment>
+<pinref part="R18" gate="G$1" pin="1"/>
+<pinref part="U1" gate="G$1" pin="GPIO2"/>
+<wire x1="106.68" y1="152.4" x2="106.68" y2="127" width="0.1524" layer="91"/>
+<wire x1="106.68" y1="127" x2="93.98" y2="127" width="0.1524" layer="91"/>
+<wire x1="106.68" y1="127" x2="119.38" y2="127" width="0.1524" layer="91"/>
+<junction x="106.68" y="127"/>
+<label x="121.92" y="127" size="1.778" layer="95"/>
 </segment>
 </net>
@@
 </segment>
 <segment>
-<wire x1="223.52" y1="167.64" x2="218.44" y2="167.64" width="0.1524" layer="91"/>
-<label x="193.04" y="167.64" size="1.778" layer="95"/>
-<pinref part="R22" gate="G$1" pin="2"/>
-<wire x1="231.14" y1="167.64" x2="223.52" y2="167.64" width="0.1524" layer="91"/>
-</segment>
-</net>
-<net name="N$22" class="0">
-<segment>
-<pinref part="JP4" gate="A" pin="1"/>
-<wire x1="243.84" y1="167.64" x2="248.92" y2="167.64" width="0.1524" layer="91"/>
-<pinref part="R22" gate="G$1" pin="1"/>
-<wire x1="241.3" y1="167.64" x2="243.84" y2="167.64" width="0.1524" layer="91"/>
+<pinref part="JP1" gate="A" pin="1"/>
+<wire x1="248.92" y1="152.4" x2="218.44" y2="152.4" width="0.1524" layer="91"/>
+<label x="198.12" y="152.4" size="1.778" layer="95"/>
 </segment>
 </net>
@@
 </segment>
 </net>
+<net name="N$24" class="0">
+<segment>
+<pinref part="R17" gate="G$1" pin="1"/>
+<pinref part="LED2" gate="G$1" pin="A"/>
+<wire x1="101.6" y1="152.4" x2="101.6" y2="149.86" width="0.1524" layer="91"/>
+</segment>
+</net>
